Commit message: Organize into gazebo and navigation

File: noob_robot_description/urdf/noob_robot.urdf.xacro (robot description, xacro)
@@ -4,5 +4,5 @@
     <xacro:property name="kinect_offset_x" value="-0.06" />
     <xacro:property name="kinect_offset_y" value="0" />
-    <xacro:property name="kinect_offset_z" value="0.055" />
+    <xacro:property name="kinect_offset_z" value="0.555" />
     <xacro:include filename="$(find noob_robot_description)/urdf/noob_robot_chassis.urdf.xacro" />
     <xacro:include filename="$(find noob_robot_description)/urdf/kinect.xacro" />

Commit message: add gmapping and configure costmap

File: noob_robot_description/urdf/noob_robot.urdf.xacro (robot description, xacro)
@@ -5,8 +5,19 @@
     <xacro:property name="kinect_offset_y" value="0" />
     <xacro:property name="kinect_offset_z" value="0.555" />
+    <!--Lidar Offset-->
+    <xacro:property name="rplidar_offset_x" value="0" />
+    <xacro:property name="rplidar_offset_y" value="0" />
+    <xacro:property name="rplidar_offset_z" value="0.04" />
     <xacro:include filename="$(find noob_robot_description)/urdf/noob_robot_chassis.urdf.xacro" />
     <xacro:include filename="$(find noob_robot_description)/urdf/kinect.xacro" />
+    <xacro:include filename="$(find noob_robot_description)/urdf/rplidar.xacro" />
     <!--Declare the xacro in the above file-->
     <xacro:noob_robot_body/>
+    <!--Laser-->
+	<joint name="rplidar_joint" type="fixed">
+		<origin xyz="${rplidar_offset_x} ${rplidar_offset_y} ${rplidar_offset_z}" rpy="0 0 0" />
+		<parent link="base_link"/>
+		<child link="laser_link"/>
+	</joint>
     <!--Kinect-->
     <joint name="kinect_frame_joint" type="fixed">
@@ -17,3 +28,4 @@
     <!--Declare the xacro in the above file-->
     <xacro:kinect_camera prefix="camera"/>
+    <xacro:rplidar prefix="laser"/>
 </robot>

File: noob_robot_description/urdf/noob_robot_chassis.urdf.xacro (robot description, xacro)
@@ -164,6 +164,6 @@
         </gazebo>
         <!-- Wheel Definitions -->
-        <xacro:wheel lr="right"  translateY="1" />
-        <xacro:wheel lr="left"  translateY="-1" />
+        <xacro:wheel lr="right"  translateY="-1" />
+        <xacro:wheel lr="left"  translateY="1" />
         <!-- Casters Definitions -->
         <xacro:caster fb="front"  translateX="-1" />
@@ -188,6 +188,6 @@
                 <wheelAcceleration>1.8</wheelAcceleration>
                 <commandTopic>cmd_vel</commandTopic>
-                <odometryFrame>gazebo_odom</odometryFrame>
-                <odometryTopic>gazebo_odom</odometryTopic>
+                <odometryFrame>odom</odometryFrame>
+                <odometryTopic>odom</odometryTopic>
                 <robotBaseFrame>base_footprint</robotBaseFrame>
             </plugin>

Commit message: fix tf issues

File: noob_robot_description/urdf/noob_robot.urdf.xacro (robot description, xacro)
@@ -17,5 +17,5 @@
 	<joint name="rplidar_joint" type="fixed">
 		<origin xyz="${rplidar_offset_x} ${rplidar_offset_y} ${rplidar_offset_z}" rpy="0 0 0" />
-		<parent link="base_link"/>
+		<parent link="base_footprint"/>
 		<child link="laser_link"/>
 	</joint>

File: noob_robot_description/urdf/noob_robot_chassis.urdf.xacro (robot description, xacro)
@@ -61,19 +61,19 @@
     </xacro:macro>
     <!-- Macro for wheel joint -->
-    <xacro:macro name="wheel" params="lr translateY">
+    <xacro:macro name="wheel" params="lr translateY">-->
         <!-- lr: left, right -->
         <link name="wheel_${lr}_link">
             <visual>
-                <origin xyz="0 0 0" rpy="${M_PI/2} 0  0 " />
+                <origin xyz="0 0 0" rpy="${M_PI/2} 0 0" />
                 <geometry>
                     <cylinder length="${wheel_height}" radius="${wheel_radius}" />
                 </geometry>
-                <material name="Blue" />
+                <material name="Red" />
             </visual>
             <collision>
-                <origin xyz="0 0 0" rpy="${M_PI/2} 0 0 " />
                 <geometry>
                     <cylinder length="${wheel_height}" radius="${wheel_radius}" />
                 </geometry>
+                <origin xyz="0 0 0" rpy="${M_PI/2} 0 0" />
             </collision>
             <xacro:cylinder_inertial_matrix  m="${wheel_mass}" r="${wheel_radius}" h="${wheel_height}" />
@@ -83,8 +83,8 @@
         </gazebo>
         <joint name="base_to_wheel_${lr}_joint" type="continuous">
-            <parent link="base_link"/>
+            <parent link="base_footprint"/>
             <child link="wheel_${lr}_link"/>
-            <origin xyz="${motor_x} ${translateY * base_link_radius} 0" rpy="0 0 0" />
-            <axis xyz="0 1 0" rpy="0  0" />
+            <origin xyz="${motor_x} ${translateY * base_link_radius} ${wheel_radius}" rpy="0 0 0" />
+            <axis xyz="0 1 0" rpy="0 0 0" />
         </joint>
         <!-- Transmission is important to link the joints and the controller -->
@@ -151,5 +151,5 @@
                     <cylinder length="${base_link_length}" radius="${base_link_radius}"/>
                 </geometry>
-                <material name="yellow" />
+                <material name="Blue" />
             </visual>
             <collision>
@@ -163,10 +163,10 @@
             <material>Gazebo/Blue</material>
         </gazebo>
+        <!-- Casters Definitions-->
+        <xacro:caster fb="front"  translateX="-1" />
+        <xacro:caster fb="back"  translateX="1" />
         <!-- Wheel Definitions -->
         <xacro:wheel lr="right"  translateY="-1" />
         <xacro:wheel lr="left"  translateY="1" />
-        <!-- Casters Definitions -->
-        <xacro:caster fb="front"  translateX="-1" />
-        <xacro:caster fb="back"  translateX="1" />
         <!-- controller -->
         <gazebo>
